File: hardware/reva/wifistepper.sch (KiCad schematic (older format))
At the start: 52 parts, among them J1 Barrel_Jack_Switch, J2 Screw_Terminal, J3 Conn_01x06, J4 Conn_01x06, J5 Conn_01x04, U1 ESP-WROOM-02, U2 powerSTEP01, U3 MAX15062A, U4 ATECC508A

Commit message: Webpage development, rework of RevA
Parts:
- removed J4: Conn_01x06, Connector_PinHeader_2.54mm:PinHeader_1x06_P2.54mm_Vertical, symbol Connector_Generic:Conn_01x06
- removed J5: Conn_01x04, Connector_PinHeader_2.54mm:PinHeader_1x04_P2.54mm_Vertical, symbol Connector_Generic:Conn_01x04
- added D0: RPOL, Klofas-Passives:D_SOD80, symbol Device:D
- added J4: Conn_01x09, Connector_PinHeader_2.54mm:PinHeader_1x09_P2.54mm_Vertical, symbol Connector_Generic:Conn_01x09
- added JP1, JP2: Jumper_2_Open, Klofas-Connectors:STpowerSTEP01_JMP, symbol Jumper:Jumper_2_Open
- added RS3, RS6: 0.06, Resistor_SMD:R_2512_6332Metric, symbol Device:R
- added SW1: SW_SPST, Klofas-Passives:TL3315NF100Q, symbol Switch:SW_SPST
- C10, C11: footprint Klofas-Passives:Capacitor_SMD-Panasonic_H13 -> Capacitor_THT:CP_Radial_D10.0mm_P5.00mm
- J2: footprint Klofas-Connectors:Phoenix_Screw_Terminal-MKDS_1,6-P3.81x06 -> TerminalBlock_Phoenix:TerminalBlock_Phoenix_PT-1,5-6-5.0-H_1x06_P5.00mm_Horizontal
- RS1: renamed from R3; value 0.2 -> 0.06
- RS2: renamed from R5; value 0.2 -> 0.06
- RS4: renamed from R4; value 0.2 -> 0.06
- RS5: renamed from R6; value 0.2 -> 0.06
Connections:
- wire segments 352 -> 372
- no-connect marks 4 -> 5
Other:
- note added: "B"
- note removed: "A"
- moved on the sheet: C21, R14, R15, RS1, RS2, RS4, RS5, U4

Commit message: Rev B design complete
Parts:
- added C22: 0.1uF, Capacitor_SMD:C_0603_1608Metric, symbol Device:C
- added J5: Conn_01x02, Connector_PinHeader_2.54mm:PinHeader_1x02_P2.54mm_Vertical, symbol Connector_Generic:Conn_01x02
Connections:
- net +3V3: now also C22.1
- net GND: now also C22.2, J5.2 (Pin_2)
- net VIN: now also J5.1 (Pin_1)
- net WIFI_ADC: now also J4.6 (Pin_6); no longer J4.5 (Pin_5)
- net WIFI_RST: now also J4.5 (Pin_5); no longer J4.6 (Pin_6)
Other:
- note added: "10/28/2018"
- note removed: "7/25/2018"
- moved on the sheet: C1, C12, C4
Changed lines of the file:
@@
 $EndComp
-$Comp
-L power:GND #PWR0101
-U 1 1 5B58D315
-P 10650 1500
-F 0 "#PWR0101" H 10650 1250 50  0001 C CNN
-F 1 "GND" H 10655 1327 50  0000 C CNN
-F 2 "" H 10650 1500 50  0001 C CNN
-F 3 "" H 10650 1500 50  0001 C CNN
-	1    10650 1500
-	1    0    0    -1
-$EndComp
-Wire Wire Line
-	10650 1500 10650 1450
-Wire Wire Line
-	10650 1450 10600 1450
-Wire Wire Line
-	10650 1250 10600 1250
 $Comp
 L Regulator_Switching:MAX15062A U3
@@
 L Device:CP C1
 U 1 1 5C91015A
-P 950 7250
-F 0 "C1" H 1068 7296 50  0000 L CNN
-F 1 "22uF" H 1068 7205 50  0000 L CNN
-F 2 "Capacitor_SMD:C_1206_3216Metric" H 988 7100 50  0001 C CNN
-F 3 "~" H 950 7250 50  0001 C CNN
-	1    950  7250
+P 750 7250
+F 0 "C1" H 868 7296 50  0000 L CNN
+F 1 "22uF" H 868 7205 50  0000 L CNN
+F 2 "Capacitor_SMD:C_1206_3216Metric" H 788 7100 50  0001 C CNN
+F 3 "~" H 750 7250 50  0001 C CNN
+	1    750  7250
 	1    0    0    -1
 $EndComp
@@
 L Device:C C4
 U 1 1 5C9102A7
-P 1400 7250
-F 0 "C4" H 1515 7296 50  0000 L CNN
-F 1 "220nF" H 1515 7205 50  0000 L CNN
-F 2 "Capacitor_SMD:C_0805_2012Metric" H 1438 7100 50  0001 C CNN
-F 3 "~" H 1400 7250 50  0001 C CNN
-	1    1400 7250
+P 1200 7250
+F 0 "C4" H 1315 7296 50  0000 L CNN
+F 1 "220nF" H 1315 7205 50  0000 L CNN
+F 2 "Capacitor_SMD:C_0805_2012Metric" H 1238 7100 50  0001 C CNN
+F 3 "~" H 1200 7250 50  0001 C CNN
+	1    1200 7250
 	1    0    0    -1
 $EndComp
@@
 L Device:C C12
 U 1 1 5C9104CA
-P 1900 7250
-F 0 "C12" H 2015 7296 50  0000 L CNN
-F 1 "0.1uF" H 2015 7205 50  0000 L CNN
-F 2 "Capacitor_SMD:C_0603_1608Metric" H 1938 7100 50  0001 C CNN
-F 3 "~" H 1900 7250 50  0001 C CNN
-	1    1900 7250
-	1    0    0    -1
-$EndComp
-Wire Wire Line
-	950  7050 950  7100
-Wire Wire Line
-	950  7400 950  7450
-Wire Wire Line
-	950  7450 1400 7450
-Wire Wire Line
-	1400 7450 1400 7400
-Wire Wire Line
-	1400 7100 1400 7050
+P 1700 7250
+F 0 "C12" H 1815 7296 50  0000 L CNN
+F 1 "0.1uF" H 1815 7205 50  0000 L CNN
+F 2 "Capacitor_SMD:C_0603_1608Metric" H 1738 7100 50  0001 C CNN
+F 3 "~" H 1700 7250 50  0001 C CNN
+	1    1700 7250
+	1    0    0    -1
+$EndComp
 Connection ~ 1400 7050
 Wire Wire Line
-	1400 7050 1900 7050
-Wire Wire Line
-	1900 7050 1900 7100
-Connection ~ 1900 7050
-Wire Wire Line
-	1900 7400 1900 7450
-Wire Wire Line
-	1900 7450 1400 7450
+	1400 7050 1700 7050
 Connection ~ 1400 7450
 $Comp
@@
 L power:+3.3V #PWR0130
 U 1 1 5CA03427
-P 900 7050
-F 0 "#PWR0130" H 900 6900 50  0001 C CNN
-F 1 "+3.3V" V 915 7178 50  0000 L CNN
-F 2 "" H 900 7050 50  0001 C CNN
-F 3 "" H 900 7050 50  0001 C CNN
-	1    900  7050
+P 650 7050
+F 0 "#PWR0130" H 650 6900 50  0001 C CNN
+F 1 "+3.3V" V 750 6950 50  0000 L CNN
+F 2 "" H 650 7050 50  0001 C CNN
+F 3 "" H 650 7050 50  0001 C CNN
+	1    650  7050
 	0    -1   -1   0
 $EndComp
-Wire Wire Line
-	900  7050 950  7050
-Connection ~ 950  7050
 Wire Wire Line
 	1400 6700 1400 6650
@@
 Wire Wire Line
 	1400 7000 1400 7050
-Wire Wire Line
-	950  7050 1400 7050
 Wire Wire Line
 	1300 6650 1400 6650
@@
 $EndComp
 $Comp
-L SparkFun-PowerSymbols:VIN #SUPPLY0104
-U 1 1 5CD08720
-P 10650 1150
-F 0 "#SUPPLY0104" H 10700 1150 45  0001 L BNN
-F 1 "VIN" H 10650 1320 45  0000 C CNN
-F 2 "XXX-00000" H 10650 1331 60  0001 C CNN
-F 3 "" H 10650 1150 60  0001 C CNN
-	1    10650 1150
-	1    0    0    -1
-$EndComp
-$Comp
 L SparkFun-PowerSymbols:VIN #SUPPLY0105
 U 1 1 5CD08856
@@
 Andrew Klofas <andrew@goodrobotics.net>
 Text Notes 8150 7650 0    50   ~ 0
-7/25/2018
+10/28/2018
 Text Notes 10600 7650 0    50   ~ 0
 B
@@
 Text GLabel 9250 5100 2    50   Input ~ 0
 WIFI_RST
-Text GLabel 10350 5350 0    50   Input ~ 0
+Text GLabel 10350 5250 0    50   Input ~ 0
 WIFI_RST
 $Comp
@@
 Text GLabel 10350 5050 0    50   Input ~ 0
 AUTH_SCK
-Text GLabel 10350 5250 0    50   Input ~ 0
+Text GLabel 10350 5350 0    50   Input ~ 0
 WIFI_ADC
 Text GLabel 9250 5000 2    50   Input ~ 0
@@
 	1    0    0    -1
 $EndComp
-Wire Wire Line
-	10650 1150 10650 1250
 NoConn ~ 10600 1350
 Wire Wire Line
@@
 Wire Wire Line
 	4200 3400 3900 3400
+$Comp
+L Device:C C22
+U 1 1 5BD3D7E2
+P 2200 7250
+F 0 "C22" H 2315 7296 50  0000 L CNN
+F 1 "0.1uF" H 2315 7205 50  0000 L CNN
+F 2 "Capacitor_SMD:C_0603_1608Metric" H 2238 7100 50  0001 C CNN
+F 3 "~" H 2200 7250 50  0001 C CNN
+	1    2200 7250
+	1    0    0    -1
+$EndComp
+Wire Wire Line
+	650  7050 750  7050
+Wire Wire Line
+	750  7100 750  7050
+Connection ~ 750  7050
+Wire Wire Line
+	750  7050 1200 7050
+Wire Wire Line
+	750  7400 750  7450
+Wire Wire Line
+	750  7450 1200 7450
+Wire Wire Line
+	1200 7100 1200 7050
+Connection ~ 1200 7050
+Wire Wire Line
+	1200 7050 1400 7050
+Wire Wire Line
+	1200 7400 1200 7450
+Connection ~ 1200 7450
+Wire Wire Line
+	1200 7450 1400 7450
+Wire Wire Line
+	1700 7450 1700 7400
+Connection ~ 1700 7450
+Wire Wire Line
+	1700 7450 1400 7450
+Wire Wire Line
+	1700 7100 1700 7050
+Connection ~ 1700 7050
+Wire Wire Line
+	1700 7050 1900 7050
+Wire Wire Line
+	1900 7050 2200 7050
+Wire Wire Line
+	2200 7050 2200 7100
+Connection ~ 1900 7050
+Wire Wire Line
+	2200 7400 2200 7450
+Wire Wire Line
+	1700 7450 2200 7450
+$Comp
+L Connector_Generic:Conn_01x02 J5
+U 1 1 5BD7FB9E
+P 10400 1900
+F 0 "J5" H 10480 1892 50  0000 L CNN
+F 1 "Conn_01x02" H 10480 1801 50  0000 L CNN
+F 2 "Connector_PinHeader_2.54mm:PinHeader_1x02_P2.54mm_Vertical" H 10400 1900 50  0001 C CNN
+F 3 "~" H 10400 1900 50  0001 C CNN
+	1    10400 1900
+	1    0    0    -1
+$EndComp
+$Comp
+L SparkFun-PowerSymbols:VIN #SUPPLY01
+U 1 1 5BD7FDCC
+P 10200 1900
+F 0 "#SUPPLY01" H 10250 1900 45  0001 L BNN
+F 1 "VIN" V 10200 2028 45  0000 L CNN
+F 2 "XXX-00000" V 10158 2028 60  0001 L CNN
+F 3 "" H 10200 1900 60  0001 C CNN
+	1    10200 1900
+	0    -1   -1   0
+$EndComp
+$Comp
+L power:GND #PWR06
+U 1 1 5BD80056
+P 10200 2000
+F 0 "#PWR06" H 10200 1750 50  0001 C CNN
+F 1 "GND" V 10205 1872 50  0000 R CNN
+F 2 "" H 10200 2000 50  0001 C CNN
+F 3 "" H 10200 2000 50  0001 C CNN
+	1    10200 2000
+	0    1    1    0
+$EndComp
+$Comp
+L SparkFun-PowerSymbols:VIN #SUPPLY02
+U 1 1 5BD80719
+P 10600 1250
+F 0 "#SUPPLY02" H 10650 1250 45  0001 L BNN
+F 1 "VIN" V 10600 1378 45  0000 L CNN
+F 2 "XXX-00000" V 10642 1378 60  0001 L CNN
+F 3 "" H 10600 1250 60  0001 C CNN
+	1    10600 1250
+	0    1    1    0
+$EndComp
+$Comp
+L power:GND #PWR07
+U 1 1 5BD809D2
+P 10600 1450
+F 0 "#PWR07" H 10600 1200 50  0001 C CNN
+F 1 "GND" V 10605 1322 50  0000 R CNN
+F 2 "" H 10600 1450 50  0001 C CNN
+F 3 "" H 10600 1450 50  0001 C CNN
+	1    10600 1450
+	0    -1   -1   0
+$EndComp
 $EndSCHEMATC
