File: hardware/wsx100/wifistepper.sch (KiCad schematic (older format))
At the start: 79 parts, among them J1 Barrel_Jack_Switch, J2 Screw_Terminal, J3 Conn_01x09, J4 Conn_01x10, J5 Conn_01x02, SW1 SW_SPST, U1 ESP-WROOM-02, U2 powerSTEP01, U3 MAX15062A, U4 ATECC508A

Commit message: final tweaks on Rev D
Parts:
- added R24, R25, R26, R27, R28: 22, Resistor_SMD:R_0603_1608Metric, symbol Device:R
- C23: value 1uF -> 0.1uF
- R1: footprint Resistor_SMD:R_0805_2012Metric_Pad1.15x1.40mm_HandSolder -> Klofas-Passives:Resistor_NP_0805
Connections:
- net AUTH_SCK: now also R27.2; no longer J4.4 (Pin_4)
- net AUTH_SDA: now also R26.2; no longer J4.3 (Pin_3)
- net PROG_BOOT: now also R28.2; no longer J4.8 (Pin_8)
- net SM_BUSY: now also R25.2; no longer J3.6 (Pin_6)
- net SM_FLAG: now also R24.2; no longer J3.5 (Pin_5)
- new net: J4.3 (Pin_3), R26.1
- new net: J4.4 (Pin_4), R27.1
- new net: J4.8 (Pin_8), R28.1
- new net: J3.5 (Pin_5), R24.1
- new net: J3.6 (Pin_6), R25.1
Other:
- moved on the sheet: R16, R17, R2
Changed lines of the file:
@@
 Text GLabel 6750 5500 0    50   Input ~ 0
 PROG_BOOT
-Text GLabel 10700 5350 0    50   Input ~ 0
+Text GLabel 10300 5350 0    50   Input ~ 0
 PROG_BOOT
 Text GLabel 10300 5550 0    50   Input ~ 0
@@
 Text GLabel 5300 1950 3    50   Input ~ 0
 SM_FLAG
-Text GLabel 10800 3200 0    50   Input ~ 0
+Text GLabel 10150 3500 0    50   Input ~ 0
 SM_FLAG
 $Comp
@@
 Wire Wire Line
 	5300 1550 5300 1500
-Text GLabel 10800 3300 0    50   Input ~ 0
+Text GLabel 10150 3600 0    50   Input ~ 0
 SM_BUSY
 $Comp
@@
 F 0 "R1" H 7720 1346 50  0000 L CNN
 F 1 "-" H 7720 1255 50  0000 L CNN
-F 2 "Resistor_SMD:R_0805_2012Metric_Pad1.15x1.40mm_HandSolder" V 7580 1300 50  0001 C CNN
+F 2 "Klofas-Passives:Resistor_NP_0805" V 7580 1300 50  0001 C CNN
 F 3 "~" H 7650 1300 50  0001 C CNN
 	1    7650 1300
@@
 Wire Wire Line
 	4650 6800 4650 6750
-Text GLabel 10700 4850 0    50   Input ~ 0
+Text GLabel 10300 4850 0    50   Input ~ 0
 AUTH_SDA
-Text GLabel 10700 4950 0    50   Input ~ 0
+Text GLabel 10300 4950 0    50   Input ~ 0
 AUTH_SCK
 Text GLabel 9600 5700 0    50   Input ~ 0
@@
 	1    0    0    -1
 $EndComp
-Text GLabel 10400 3400 0    50   Input ~ 0
+Text GLabel 10250 3750 0    50   Input ~ 0
 SM_CLK
-Text GLabel 10400 3600 0    50   Input ~ 0
+Text GLabel 10250 3950 0    50   Input ~ 0
 SM_SO
-Text GLabel 10400 3500 0    50   Input ~ 0
+Text GLabel 10250 3850 0    50   Input ~ 0
 SM_SI
 Wire Wire Line
@@
 L Device:R R2
 U 1 1 5C50BF9F
-P 10550 3600
-F 0 "R2" V 10600 3800 50  0000 C CNN
-F 1 "22" V 10550 3600 50  0000 C CNN
-F 2 "Resistor_SMD:R_0603_1608Metric" V 10480 3600 50  0001 C CNN
-F 3 "~" H 10550 3600 50  0001 C CNN
-	1    10550 3600
+P 10400 3950
+F 0 "R2" V 10450 4150 50  0000 C CNN
+F 1 "22" V 10400 3950 50  0000 C CNN
+F 2 "Resistor_SMD:R_0603_1608Metric" V 10330 3950 50  0001 C CNN
+F 3 "~" H 10400 3950 50  0001 C CNN
+	1    10400 3950
 	0    1    1    0
 $EndComp
@@
 L Device:R R16
 U 1 1 5C5B87C0
-P 10550 3400
-F 0 "R16" V 10600 3600 50  0000 C CNN
-F 1 "22" V 10550 3400 50  0000 C CNN
-F 2 "Resistor_SMD:R_0603_1608Metric" V 10480 3400 50  0001 C CNN
-F 3 "~" H 10550 3400 50  0001 C CNN
-	1    10550 3400
+P 10400 3750
+F 0 "R16" V 10450 3950 50  0000 C CNN
+F 1 "22" V 10400 3750 50  0000 C CNN
+F 2 "Resistor_SMD:R_0603_1608Metric" V 10330 3750 50  0001 C CNN
+F 3 "~" H 10400 3750 50  0001 C CNN
+	1    10400 3750
 	0    1    1    0
 $EndComp
@@
 L Device:R R17
 U 1 1 5C5B8DA2
-P 10550 3500
-F 0 "R17" V 10600 3700 50  0000 C CNN
-F 1 "22" V 10550 3500 50  0000 C CNN
-F 2 "Resistor_SMD:R_0603_1608Metric" V 10480 3500 50  0001 C CNN
-F 3 "~" H 10550 3500 50  0001 C CNN
-	1    10550 3500
+P 10400 3850
+F 0 "R17" V 10450 4050 50  0000 C CNN
+F 1 "22" V 10400 3850 50  0000 C CNN
+F 2 "Resistor_SMD:R_0603_1608Metric" V 10330 3850 50  0001 C CNN
+F 3 "~" H 10400 3850 50  0001 C CNN
+	1    10400 3850
 	0    1    1    0
 $EndComp
@@
 U 1 1 5CEA01A4
 P 10450 5250
-F 0 "R19" V 10400 5450 50  0000 C CNN
+F 0 "R19" V 10500 5450 50  0000 C CNN
 F 1 "22" V 10450 5250 50  0000 C CNN
 F 2 "Resistor_SMD:R_0603_1608Metric" V 10380 5250 50  0001 C CNN
@@
 U 1 1 5CF5D1C1
 P 9900 3250
-F 0 "C24" V 10150 3250 50  0000 C CNN
-F 1 "0.1uF" V 10050 3250 50  0000 C CNN
+F 0 "C24" V 10050 3250 50  0000 C CNN
+F 1 "0.1uF" V 9950 3400 50  0000 C CNN
 F 2 "Capacitor_SMD:C_0603_1608Metric" H 9938 3100 50  0001 C CNN
 F 3 "~" H 9900 3250 50  0001 C CNN
@@
 P 9900 2850
 F 0 "C23" V 9648 2850 50  0000 C CNN
-F 1 "1uF" V 9739 2850 50  0000 C CNN
+F 1 "0.1uF" V 9739 2850 50  0000 C CNN
 F 2 "Capacitor_SMD:C_0603_1608Metric" H 9938 2700 50  0001 C CNN
 F 3 "~" H 9900 2850 50  0001 C CNN
@@
 	10700 3500 10800 3500
 Wire Wire Line
-	10700 3600 10800 3600
-Wire Wire Line
 	10600 5550 10700 5550
-Wire Wire Line
-	10700 3400 10800 3400
 $Comp
 L Device:D_Schottky D0
@@
 	-1   0    0    1
 $EndComp
+$Comp
+L Device:R R27
+U 1 1 5C5D5808
+P 10450 4950
+F 0 "R27" V 10500 5150 50  0000 C CNN
+F 1 "22" V 10450 4950 50  0000 C CNN
+F 2 "Resistor_SMD:R_0603_1608Metric" V 10380 4950 50  0001 C CNN
+F 3 "~" H 10450 4950 50  0001 C CNN
+	1    10450 4950
+	0    1    1    0
+$EndComp
+$Comp
+L Device:R R26
+U 1 1 5C5D58BC
+P 10450 4850
+F 0 "R26" V 10500 5050 50  0000 C CNN
+F 1 "22" V 10450 4850 50  0000 C CNN
+F 2 "Resistor_SMD:R_0603_1608Metric" V 10380 4850 50  0001 C CNN
+F 3 "~" H 10450 4850 50  0001 C CNN
+	1    10450 4850
+	0    1    1    0
+$EndComp
+Wire Wire Line
+	10750 3600 10800 3600
+Wire Wire Line
+	10650 3400 10800 3400
+$Comp
+L Device:R R25
+U 1 1 5C7B0008
+P 10300 3600
+F 0 "R25" V 10350 3800 50  0000 C CNN
+F 1 "22" V 10300 3600 50  0000 C CNN
+F 2 "Resistor_SMD:R_0603_1608Metric" V 10230 3600 50  0001 C CNN
+F 3 "~" H 10300 3600 50  0001 C CNN
+	1    10300 3600
+	0    1    1    0
+$EndComp
+$Comp
+L Device:R R24
+U 1 1 5C7DFA3D
+P 10300 3500
+F 0 "R24" V 10350 3700 50  0000 C CNN
+F 1 "22" V 10300 3500 50  0000 C CNN
+F 2 "Resistor_SMD:R_0603_1608Metric" V 10230 3500 50  0001 C CNN
+F 3 "~" H 10300 3500 50  0001 C CNN
+	1    10300 3500
+	0    1    1    0
+$EndComp
+Wire Wire Line
+	10800 3300 10600 3300
+Wire Wire Line
+	10600 3300 10600 3600
+Wire Wire Line
+	10600 3600 10450 3600
+Wire Wire Line
+	10800 3200 10550 3200
+Wire Wire Line
+	10550 3200 10550 3500
+Wire Wire Line
+	10550 3500 10450 3500
+Wire Wire Line
+	10550 3750 10650 3750
+Wire Wire Line
+	10650 3400 10650 3750
+Wire Wire Line
+	10550 3850 10700 3850
+Wire Wire Line
+	10700 3500 10700 3850
+Wire Wire Line
+	10550 3950 10750 3950
+Wire Wire Line
+	10750 3600 10750 3950
+Wire Wire Line
+	10600 4850 10700 4850
+Wire Wire Line
+	10700 4950 10600 4950
+$Comp
+L Device:R R28
+U 1 1 5C999B8B
+P 10450 5350
+F 0 "R28" V 10500 5550 50  0000 C CNN
+F 1 "22" V 10450 5350 50  0000 C CNN
+F 2 "Resistor_SMD:R_0603_1608Metric" V 10380 5350 50  0001 C CNN
+F 3 "~" H 10450 5350 50  0001 C CNN
+	1    10450 5350
+	0    1    1    0
+$EndComp
+Wire Wire Line
+	10600 5350 10700 5350
 $EndSCHEMATC

Commit message: Updated board layout
Parts:
- removed J3: Conn_01x09, Connector_PinHeader_2.54mm:PinHeader_1x09_P2.54mm_Vertical, symbol Connector_Generic:Conn_01x09
- added D7: 50V Clamp, Klofas-Passives:D_SMF_DO-219AB, symbol Device:D_Zener
- added J3: Conn_01x10, Connector_PinHeader_2.54mm:PinHeader_1x10_P2.54mm_Vertical, symbol Connector_Generic:Conn_01x10
- added R29: 22, Resistor_SMD:R_0603_1608Metric, symbol Device:R
- D0: footprint Diode_SMD:D_SOD-123F -> Diode_SMD:D_SMB
Connections:
- net +3V3: now also J3.1 (Pin_1)
- net GND: now also D7.2 (A), J3.2 (Pin_2)
- net SM_CS: now also R29.2
- net at C18.1, JP0.2 (B), U3.1 (VIN)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: now also D7.1 (K)
- net at R22.1: now also J3.3 (Pin_3)
- net at R23.1: now also J3.4 (Pin_4)
- net at R24.1: now also J3.5 (Pin_5)
- net at R25.1: now also J3.6 (Pin_6)
- net at R16.1: now also J3.7 (Pin_7)
- net at R17.1: now also J3.8 (Pin_8)
- net at R2.1: now also J3.9 (Pin_9)
- new net: J3.10 (Pin_10), R29.1
Other:
- moved on the sheet: C18, FB1, JP0, R16, R17, R2, R24, R25
